File: SOCSchem/SOCSchem.sch (KiCad schematic (older format))
At the start: 26 parts

Commit message: Lots of bug fixes and added JALR/JAL
Parts:
- removed U?: PC, symbol SOC:PC
- removed U?: ID_IE, symbol SOC:ID-IE
- removed U?: REGFILE, symbol SOC:REGFILE
- removed U?: IMM_GEN, symbol SOC:IMM_GEN
- removed U?: IE_MEM, symbol SOC:IE-MEM
- removed U?: WB-MUX, symbol SOC:WB-MUX
- removed U?: DECODER, symbol SOC:DECODER
- removed U?: IF_ID, symbol SOC:IF-ID
- removed U? (x2): 3-1MUX, symbol SOC:3-1MUX
- removed U?: DBUS, symbol SOC:DBUS
- removed U?: PC_ADDER, symbol SOC:ADDER
- removed U? (x5): 2-1Mux, symbol SOC:2-1Mux
- removed U?: IRAM, symbol SOC:IRAM
- removed U?: FORWARDING_UNIT, symbol SOC:FORWARDING_UNIT
- removed U?: BRANCH_ADDER, symbol SOC:ADDER
- removed U?: BRANCH_UNIT, symbol SOC:BRANCH_UNIT
- removed U?: MATH_UNIT, symbol SOC:MATH_UNIT
- removed U?: BARREL_SHIFTER, symbol SOC:BARREL_SHIFTER
- removed U?: HAZARD_UNIT, symbol SOC:HAZARD_UNIT
- removed U?: 0Comparator, symbol SOC:0Comparator
- removed U?: MEM-WB, symbol SOC:MEM-WB
- added U?: ARBITER, symbol SOC:ARBITER
Connections:
- net labels added: DBUS_Gnt, DBUS_Req
- net labels removed: 4, AluBSel_E, AluForASel, AluForBSel, AluRes_M, AluRes_W, AluZero_M, Clr_D, Clr_E, Clr_M, Clr_W, DBusForASel, DBusForBSel, DRamWe_M, En_D, En_E, En_M, En_W, Func3_E, Func3_M, IRamOZero, IRamRdEn, Imm_M, Immediate_E, Inst[11:7], Inst[19:15], Inst[24:20], IsBranch_E, IsBranch_M, PC_E, PC_F, PC_M, PcEn, RDAddr_D, RDAddr_E, RDAddr_M, RDAddr_W, RS1Addr_D, RS1Addr_E, RS1_D, RS2Addr_D, RS2Addr_E, RS2Addr_M, RS2_D, RS2_E, RegWrEn_M, RegWrEn_W, TakeBranch, TakeBranch_M, WBData_W, WBSrc_E, WBSrc_M, WBSrc_W
- wire segments 141 -> 0

Commit message: Various improvments and fixes
Parts:
- removed U?: ARBITER, symbol SOC:ARBITER
Connections:
- net labels removed: DBUS_Gnt, DBUS_Req
Changed lines of the file:
@@
 $Descr A4 11693 8268
 encoding utf-8
-Sheet 1 2
+Sheet 1 1
 Title ""
 Date ""
@@
 Comment4 ""
 $EndDescr
-$Sheet
-S 9775 700  975  750
-U 5EB97B98
-F0 "CPU" 39
-F1 "CPU.sch" 39
-F2 "DBUS_Addr" O L 9775 950 50
-F3 "DBUS_ByteEn" O L 9775 1025 50
-F4 "DBUS_Read" O L 9775 1100 50
-F5 "DBUS_Write" O L 9775 1175 50
-F6 "DBUS_Rd" I L 9775 1250 50
-F7 "DBUS_Wd" O L 9775 1325 50
-F8 "DBUS_Req" O L 9775 750 50
-F9 "DBUS_Gnt" I L 9775 825 50
-F10 "DBUS_WaitReq" I L 9775 1400 50
-$EndSheet
-$Comp
-L SOC:ARBITER U?
-U 1 1 5EBABA86
-P 8325 750
-F 0 "U?" H 8400 1150 31  0001 C CNN
-F 1 "ARBITER" H 8350 850 39  0000 C CNN
-F 2 "" H 8400 1150 31  0001 C CNN
-F 3 "" H 8400 1150 31  0001 C CNN
-	1    8325 750
-	1    0    0    -1
-$EndComp
-Text Label 9775 750  2    39   ~ 0
-DBUS_Req
-Text Label 9775 825  2    39   ~ 0
-DBUS_Gnt
-Text Label 8175 750  2    39   ~ 0
-DBUS_Req
-Text Label 8600 750  0    39   ~ 0
-DBUS_Gnt
 $EndSCHEMATC
